Commit message: [Change] arm joint defination

File: tinker_description/urdf/arm/arm.urdf.xacro (robot description, xacro)
@@ -4,9 +4,15 @@
     <xacro:property name="arm_origin_y" value="0"/>
     <xacro:property name="arm_origin_z" value="0.77"/>
-    <joint name="arm_origin_joint" type="prismatic">
+    <joint name="arm_origin_joint" type="fixed">
+        <parent link="base_link"/>
+        <child link="arm_origin_link"/>
+        <origin xyz="${arm_origin_x} ${arm_origin_y} ${arm_origin_z}" rpy="0 0 0"/>
+    </joint>
+    <link name="arm_origin_link"/>
+    <joint name="arm_base_joint" type="prismatic">
         <axis xyz="0 0 1"/>
-        <parent link="base_link"/>
+        <parent link="arm_origin_link"/>
         <child link="arm_base_link"/>
-        <origin xyz="${arm_origin_x} ${arm_origin_y} ${arm_origin_z}" rpy="0 0 0"/>
+        <origin xyz="0 0 0" rpy="0 0 0"/>
         <limit effort="1000.0" lower="0" upper="0.4" velocity="0.5"/>
     </joint>
@@ -58,6 +64,6 @@
         <parent link="shoulder_base_link"/>
         <child link="shoulder_link"/>
-        <limit effort="1000.0" lower="0" upper="${M_PI/4}" velocity="0.5"/>
-        <origin xyz="0 0 0.1" rpy="0 0 0"/>
+        <limit effort="1000.0" lower="0" upper="${M_PI/2}" velocity="0.5"/>
+        <origin xyz="0 0 0.1" rpy="${-M_PI/2} 0 ${M_PI}"/>
     </joint>
     <link name="shoulder_link">
@@ -84,6 +90,6 @@
         <parent link="shoulder_link"/>
         <child link="elbow_link"/>
-        <limit effort="1000.0" lower="${M_PI/6}" upper="${M_PI}" velocity="0.5"/>
-        <origin xyz="0 0 0.34" rpy="0 ${M_PI} 0"/>
+        <limit effort="1000.0" lower="0" upper="${M_PI}" velocity="0.5"/>
+        <origin xyz="0 0 0.34" rpy="0 0 ${M_PI}"/>
     </joint>
     <link name="elbow_link">
@@ -106,10 +112,10 @@
         </inertial>
     </link>
-    <joint name="wrist_deviation_joint" type="revolute">
+    <joint name="wrist_deviation" type="revolute">
         <axis xyz="0 1 0"/>
         <parent link="elbow_link"/>
         <child link="wrist_deviation_link"/>
-        <limit effort="1000.0" lower="${-M_PI/2}" upper="${M_PI/2}" velocity="0.5"/>
-        <origin xyz="0 0 0.34" rpy="0 0 0"/>
+        <limit effort="1000.0" lower="${M_PI/2}" upper="${M_PI*3/2}" velocity="0.5"/>
+        <origin xyz="0 0 0.34" rpy="${M_PI} 0 ${M_PI}"/>
     </joint>
     <link name="wrist_deviation_link">
@@ -132,10 +138,10 @@
         </inertial>
     </link>
-    <joint name="wrist_extension_joint" type="revolute">
+    <joint name="wrist_extension" type="revolute">
         <axis xyz="1 0 0"/>
         <parent link="wrist_deviation_link"/>
         <child link="wrist_extension_link"/>
-        <limit effort="1000.0" lower="${-M_PI/2}" upper="${M_PI/2}" velocity="0.5"/>
-        <origin xyz="0 0 0.1" rpy="0 0 0"/>
+        <limit effort="1000.0" lower="${M_PI/2}" upper="${M_PI*3/2}" velocity="0.5"/>
+        <origin xyz="0 0 0.1" rpy="0 ${M_PI} 0"/>
     </joint>
     <link name="wrist_extension_link">
@@ -158,5 +164,5 @@
         </inertial>
     </link>
-    <xacro:pr2_gripper_v0 reflect="-1.0" side="" parent="wrist_extension_link"
+    <!--xacro:pr2_gripper_v0 reflect="-1.0" side="" parent="wrist_extension_link"
         screw_reduction="${4.0/1000.0}"
         gear_ratio="${(729.0/25.0)*(22.0/16.0)}"
@@ -170,4 +176,4 @@
         r="${91.5/1000.0}">
         <origin xyz="0 0 0.08" rpy="0 ${-M_PI/2} ${M_PI/2}" />
-    </xacro:pr2_gripper_v0>
+    </xacro:pr2_gripper_v0-->
 </robot>

Commit message: [Change] tinker description

File: tinker_description/urdf/arm/arm.urdf.xacro (robot description, xacro)
@@ -3,5 +3,5 @@
     <xacro:property name="arm_origin_x" value="0.12"/>
     <xacro:property name="arm_origin_y" value="0"/>
-    <xacro:property name="arm_origin_z" value="0.54"/>
+    <xacro:property name="arm_origin_z" value="0.69"/>
     <xacro:property name="shoulder_base_link_length" value="0.06"/>
     <xacro:property name="shoulder_link_length" value="0.41"/>

File: tinker_description/urdf/body/body.urdf.xacro (robot description, xacro)
@@ -31,5 +31,5 @@
     <xacro:include filename="$(find pr2_description)/urdf/sensors/kinect2.urdf.xacro"/>
     <xacro:kinect2_v0 name="kinect" parent="pillar">
-        <origin xyz="0.06 0 0.9" rpy="0 0 0"/>
+        <origin xyz="0.06 0.05 0.98" rpy="0 0 0"/>
     </xacro:kinect2_v0>
 </robot>

Commit message: [Change] arm origin pos

File: tinker_description/urdf/arm/arm.urdf.xacro (robot description, xacro)
@@ -1,7 +1,7 @@
 <?xml version="1.0"?>
 <robot xmlns:xacro="http://ros.org/wiki/xacro">
-    <xacro:property name="arm_origin_x" value="0.12"/>
-    <xacro:property name="arm_origin_y" value="0"/>
-    <xacro:property name="arm_origin_z" value="0.69"/>
+    <xacro:property name="arm_origin_x" value="0.15"/>
+    <xacro:property name="arm_origin_y" value="-0.06"/>
+    <xacro:property name="arm_origin_z" value="0.71"/>
     <xacro:property name="shoulder_base_link_length" value="0.06"/>
     <xacro:property name="shoulder_link_length" value="0.41"/>

File: tinker_description/urdf/base/base.urdf.xacro (robot description, xacro)
@@ -9,5 +9,5 @@
     <xacro:property name="base_width" value="0.52"/>
     <xacro:property name="base_height" value="0.18"/>
-    <xacro:property name="base_laser_x" value="0.30"/>
+    <xacro:property name="base_laser_x" value="0.0"/>
     <xacro:property name="base_laser_y" value="0"/>
     <xacro:property name="base_laser_z" value="0.185"/>

Commit message: Robocup 2016

File: tinker_description/urdf/arm/arm.urdf.xacro (robot description, xacro)
@@ -2,5 +2,5 @@
 <robot xmlns:xacro="http://ros.org/wiki/xacro">
     <xacro:property name="arm_origin_x" value="0.15"/>
-    <xacro:property name="arm_origin_y" value="-0.06"/>
+    <xacro:property name="arm_origin_y" value="-0.09"/>
     <xacro:property name="arm_origin_z" value="0.71"/>
     <xacro:property name="shoulder_base_link_length" value="0.06"/>

File: tinker_description/urdf/body/body.urdf.xacro (robot description, xacro)
@@ -31,5 +31,5 @@
     <xacro:include filename="$(find pr2_description)/urdf/sensors/kinect2.urdf.xacro"/>
     <xacro:kinect2_v0 name="kinect" parent="pillar">
-        <origin xyz="0.06 0.05 0.98" rpy="0 0 0"/>
+        <origin xyz="0.06 0.05 1.00" rpy="0 0 0"/>
     </xacro:kinect2_v0>
 </robot>
