Commit message: [Add] New primesense sensors description

File: tinker_description/urdf/base/base.urdf.xacro (robot description, xacro)
@@ -6,4 +6,5 @@
     <xacro:include filename="$(find tinker_description)/urdf/base/base.gazebo.xacro"/>
     <xacro:include filename="$(find tinker_description)/urdf/sensor/hokuyo_lx30_laser.urdf.xacro"/>
+    <xacro:include filename="$(find hector_sensors_description)/urdf/realsense_camera.urdf.xacro"/>
     <xacro:property name="base_length" value="0.64"/>
     <xacro:property name="base_width" value="0.52"/>
@@ -11,5 +12,11 @@
     <xacro:property name="base_laser_x" value="0.30"/>
     <xacro:property name="base_laser_y" value="0"/>
-    <xacro:property name="base_laser_z" value="0.185"/>
+    <xacro:property name="base_laser_z" value="0.25"/>
+    <xacro:property name="front_primesense_x" value="0.30"/>
+    <xacro:property name="front_primesense_y" value="0"/>
+    <xacro:property name="front_primesense_z" value="0.1"/>
+    <xacro:property name="back_xtion_x" value="-0.30"/>
+    <xacro:property name="back_xtion_y" value="0"/>
+    <xacro:property name="back_xtion_z" value="0.1"/>
     <!--*****************chasiss***********************-->
     <link name="base_link">
@@ -37,3 +44,9 @@
         <origin xyz="${base_laser_x} ${base_laser_y} ${base_laser_z}" rpy="0 0 0"/>
     </xacro:hokuyo_lx30_laser_v0>
+    <xacro:realsense_camera name="primesense_front" parent="base_link">
+        <origin xyz="${front_primesense_x} ${front_primesense_y} ${front_primesense_z}" rpy="0 0 0"/>
+    </xacro:realsense_camera>
+    <xacro:realsense_camera name="xtion_back" parent="base_link">
+        <origin xyz="${back_xtion_x} ${back_xtion_y} ${back_xtion_z}" rpy="0 0 ${M_PI}"/>
+    </xacro:realsense_camera>
 </robot>

Commit message: [Fix] Remove laptop from tinker machine

File: tinker_description/urdf/base/base.urdf.xacro (robot description, xacro)
@@ -10,8 +10,8 @@
     <xacro:property name="base_width" value="0.52"/>
     <xacro:property name="base_height" value="0.18"/>
-    <xacro:property name="base_laser_x" value="0.0"/>
+    <xacro:property name="base_laser_x" value="0.30"/>
     <xacro:property name="base_laser_y" value="0"/>
     <xacro:property name="base_laser_z" value="0.25"/>
-    <xacro:property name="front_primesense_x" value="0.30"/>
+    <xacro:property name="front_primesense_x" value="0.40"/>
     <xacro:property name="front_primesense_y" value="0"/>
     <xacro:property name="front_primesense_z" value="0.1"/>
