Commit message: [ADD] arm description

File: tinker_description/robot/tinker.urdf.xacro (robot description, xacro)
@@ -6,4 +6,5 @@
        name="tinker">
     <xacro:include filename="$(find pr2_description)/urdf/common.xacro"/>
+    <xacro:include filename="$(find pr2_description)/urdf/gripper_v0/gripper.urdf.xacro" />
     <xacro:include filename="$(find tinker_description)/urdf/materials.xacro"/>
     <xacro:include filename="$(find tinker_description)/urdf/base/base.urdf.xacro"/>

File: tinker_description/urdf/arm/arm.urdf.xacro (robot description, xacro)
@@ -4,8 +4,15 @@
     <xacro:property name="arm_origin_y" value="0"/>
     <xacro:property name="arm_origin_z" value="0.77"/>
-    <link name="arm_link">
+    <joint name="arm_origin_joint" type="prismatic">
+        <axis xyz="0 0 1"/>
+        <parent link="base_link"/>
+        <child link="arm_base_link"/>
+        <origin xyz="${arm_origin_x} ${arm_origin_y} ${arm_origin_z}" rpy="0 0 0"/>
+        <limit effort="1000.0" lower="0" upper="0.4" velocity="0.5"/>
+    </joint>
+    <link name="arm_base_link">
         <visual>
             <geometry>
-                <box size="0.2 0.1 0.03"/>
+                <box size="0.1 0.1 0.04"/>
             </geometry>
             <material name="green"/>
@@ -13,5 +20,5 @@
         <collision>
             <geometry>
-                <box size="0.2 0.1 0.03"/>
+                <box size="0.1 0.1 0.04"/>
             </geometry>
         </collision>
@@ -21,10 +28,146 @@
         </inertial>
     </link>
-    <joint name="arm_origin_joint" type="prismatic">
+    <joint name="shoulder_rotation_joint" type="revolute">
         <axis xyz="0 0 1"/>
-        <parent link="base_link"/>
-        <child link="arm_link"/>
-        <origin xyz="${arm_origin_x} ${arm_origin_y} ${arm_origin_z}" rpy="0 0 0"/>
-        <limit effort="1000.0" lower="0" upper="0.5" velocity="0.5"/>
+        <parent link="arm_base_link"/>
+        <child link="shoulder_base_link"/>
+        <limit effort="1000.0" lower="${-M_PI/2}" upper="${M_PI/2}" velocity="0.5"/>
+        <origin xyz="0 0 0" rpy="0 0 ${M_PI/2}"/>
     </joint>
+    <link name="shoulder_base_link">
+        <visual>
+            <geometry>
+                <cylinder length="0.1" radius="0.04"/>
+            </geometry>
+            <origin xyz="0 0 0.05" rpy="0 0 ${M_PI}"/>
+            <material name="red"/>
+        </visual>
+        <collision>
+            <geometry>
+                <cylinder length="0.1" radius="0.04"/>
+            </geometry>
+            <origin xyz="0 0 0.05" rpy="0 0 ${M_PI}"/>
+        </collision>
+        <inertial>
+            <mass value="1"/>
+            <inertia ixx="0.0" ixy="0.0" ixz="0.0" iyy="0.0" iyz="0.0" izz="0.0"/>
+        </inertial>
+    </link>
+    <joint name="shoulder_flexion_joint" type="revolute">
+        <axis xyz="1 0 0"/>
+        <parent link="shoulder_base_link"/>
+        <child link="shoulder_link"/>
+        <limit effort="1000.0" lower="0" upper="${M_PI/4}" velocity="0.5"/>
+        <origin xyz="0 0 0.1" rpy="0 0 0"/>
+    </joint>
+    <link name="shoulder_link">
+        <visual>
+            <geometry>
+                <cylinder length="0.34" radius="0.04"/>
+            </geometry>
+            <origin xyz="0 0 0.17" rpy="0 0 0"/>
+            <material name="blue"/>
+        </visual>
+        <collision>
+            <geometry>
+                <cylinder length="0.34" radius="0.04"/>
+            </geometry>
+            <origin xyz="0 0 0.17" rpy="0 0 0"/>
+        </collision>
+        <inertial>
+            <mass value="1"/>
+            <inertia ixx="0.0" ixy="0.0" ixz="0.0" iyy="0.0" iyz="0.0" izz="0.0"/>
+        </inertial>
+    </link>
+    <joint name="elbow_joint" type="revolute">
+        <axis xyz="1 0 0"/>
+        <parent link="shoulder_link"/>
+        <child link="elbow_link"/>
+        <limit effort="1000.0" lower="${M_PI/6}" upper="${M_PI}" velocity="0.5"/>
+        <origin xyz="0 0 0.34" rpy="0 ${M_PI} 0"/>
+    </joint>
+    <link name="elbow_link">
+        <visual>
+            <geometry>
+                <cylinder length="0.34" radius="0.04"/>
+            </geometry>
+            <origin xyz="0 0 0.17" rpy="0 0 0"/>
+            <material name="white"/>
+        </visual>
+        <collision>
+            <geometry>
+                <cylinder length="0.34" radius="0.04"/>
+            </geometry>
+            <origin xyz="0 0 0.17" rpy="0 0 0"/>
+        </collision>
+        <inertial>
+            <mass value="1"/>
+            <inertia ixx="0.0" ixy="0.0" ixz="0.0" iyy="0.0" iyz="0.0" izz="0.0"/>
+        </inertial>
+    </link>
+    <joint name="wrist_deviation_joint" type="revolute">
+        <axis xyz="0 1 0"/>
+        <parent link="elbow_link"/>
+        <child link="wrist_deviation_link"/>
+        <limit effort="1000.0" lower="${-M_PI/2}" upper="${M_PI/2}" velocity="0.5"/>
+        <origin xyz="0 0 0.34" rpy="0 0 0"/>
+    </joint>
+    <link name="wrist_deviation_link">
+        <visual>
+            <geometry>
+                <cylinder length="0.10" radius="0.04"/>
+            </geometry>
+            <origin xyz="0 0 0.05" rpy="0 0 0"/>
+            <material name="green"/>
+        </visual>
+        <collision>
+            <geometry>
+                <cylinder length="0.10" radius="0.04"/>
+            </geometry>
+            <origin xyz="0 0 0.5" rpy="0 0 0"/>
+        </collision>
+        <inertial>
+            <mass value="1"/>
+            <inertia ixx="0.0" ixy="0.0" ixz="0.0" iyy="0.0" iyz="0.0" izz="0.0"/>
+        </inertial>
+    </link>
+    <joint name="wrist_extension_joint" type="revolute">
+        <axis xyz="1 0 0"/>
+        <parent link="wrist_deviation_link"/>
+        <child link="wrist_extension_link"/>
+        <limit effort="1000.0" lower="${-M_PI/2}" upper="${M_PI/2}" velocity="0.5"/>
+        <origin xyz="0 0 0.1" rpy="0 0 0"/>
+    </joint>
+    <link name="wrist_extension_link">
+        <visual>
+            <geometry>
+                <cylinder length="0.10" radius="0.04"/>
+            </geometry>
+            <origin xyz="0 0 0.05" rpy="0 0 0"/>
+            <material name="blue"/>
+        </visual>
+        <collision>
+            <geometry>
+                <cylinder length="0.10" radius="0.04"/>
+            </geometry>
+            <origin xyz="0 0 0.5" rpy="0 0 0"/>
+        </collision>
+        <inertial>
+            <mass value="1"/>
+            <inertia ixx="0.0" ixy="0.0" ixz="0.0" iyy="0.0" iyz="0.0" izz="0.0"/>
+        </inertial>
+    </link>
+    <xacro:pr2_gripper_v0 reflect="-1.0" side="" parent="wrist_extension_link"
+        screw_reduction="${4.0/1000.0}"
+        gear_ratio="${(729.0/25.0)*(22.0/16.0)}"
+        theta0="${3.6029*M_PI/180.0}"
+        phi0="${29.7089*M_PI/180.0}"
+        t0="${-0.1914/1000.0}"
+        L0="${37.5528/1000.0}"
+        h="${0.0/1000.0}"
+        a="${68.3698/1000.0}"
+        b="${43.3849/1000.0}"
+        r="${91.5/1000.0}">
+        <origin xyz="0 0 0.08" rpy="0 ${-M_PI/2} ${M_PI/2}" />
+    </xacro:pr2_gripper_v0>
 </robot>

Commit message: [Change] arm & kinect position

File: tinker_description/robot/tinker.urdf.xacro (robot description, xacro)
@@ -6,5 +6,4 @@
        name="tinker">
     <xacro:include filename="$(find pr2_description)/urdf/common.xacro"/>
-    <xacro:include filename="$(find pr2_description)/urdf/gripper_v0/gripper.urdf.xacro" />
     <xacro:include filename="$(find tinker_description)/urdf/materials.xacro"/>
     <xacro:include filename="$(find tinker_description)/urdf/base/base.urdf.xacro"/>

File: tinker_description/urdf/arm/arm.urdf.xacro (robot description, xacro)
@@ -3,5 +3,10 @@
     <xacro:property name="arm_origin_x" value="0.12"/>
     <xacro:property name="arm_origin_y" value="0"/>
-    <xacro:property name="arm_origin_z" value="0.77"/>
+    <xacro:property name="arm_origin_z" value="0.54"/>
+    <xacro:property name="shoulder_base_link_length" value="0.06"/>
+    <xacro:property name="shoulder_link_length" value="0.41"/>
+    <xacro:property name="elbow_link_length" value="0.32"/>
+    <xacro:property name="wrist_deviation_link_length" value="0.09"/>
+    <xacro:property name="wrist_extension_link_length" value="0.10"/>
     <joint name="arm_origin_joint" type="fixed">
         <parent link="base_link"/>
@@ -44,14 +49,14 @@
         <visual>
             <geometry>
-                <cylinder length="0.1" radius="0.04"/>
+                <cylinder length="${shoulder_base_link_length}" radius="0.04"/>
             </geometry>
-            <origin xyz="0 0 0.05" rpy="0 0 ${M_PI}"/>
+            <origin xyz="0 0 ${shoulder_base_link_length/2}" rpy="0 0 ${M_PI}"/>
             <material name="red"/>
         </visual>
         <collision>
             <geometry>
-                <cylinder length="0.1" radius="0.04"/>
+                <cylinder length="${shoulder_base_link_length}" radius="0.04"/>
             </geometry>
-            <origin xyz="0 0 0.05" rpy="0 0 ${M_PI}"/>
+            <origin xyz="0 0 ${shoulder_base_link_length/2}" rpy="0 0 ${M_PI}"/>
         </collision>
         <inertial>
@@ -65,19 +70,19 @@
         <child link="shoulder_link"/>
         <limit effort="1000.0" lower="0" upper="${M_PI/2}" velocity="0.5"/>
-        <origin xyz="0 0 0.1" rpy="${-M_PI/2} 0 ${M_PI}"/>
+        <origin xyz="0 0 ${shoulder_base_link_length}" rpy="${-M_PI/2} 0 ${M_PI}"/>
     </joint>
     <link name="shoulder_link">
         <visual>
             <geometry>
-                <cylinder length="0.34" radius="0.04"/>
+                <cylinder length="${shoulder_link_length}" radius="0.04"/>
             </geometry>
-            <origin xyz="0 0 0.17" rpy="0 0 0"/>
+            <origin xyz="0 0 ${shoulder_link_length/2}" rpy="0 0 0"/>
             <material name="blue"/>
         </visual>
         <collision>
             <geometry>
-                <cylinder length="0.34" radius="0.04"/>
+                <cylinder length="${shoulder_link_length}" radius="0.04"/>
             </geometry>
-            <origin xyz="0 0 0.17" rpy="0 0 0"/>
+            <origin xyz="0 0 ${shoulder_link_length/2}" rpy="0 0 0"/>
         </collision>
         <inertial>
@@ -91,19 +96,19 @@
         <child link="elbow_link"/>
         <limit effort="1000.0" lower="0" upper="${M_PI}" velocity="0.5"/>
-        <origin xyz="0 0 0.34" rpy="0 0 ${M_PI}"/>
+        <origin xyz="0 0 ${shoulder_link_length}" rpy="0 0 ${M_PI}"/>
     </joint>
     <link name="elbow_link">
         <visual>
             <geometry>
-                <cylinder length="0.34" radius="0.04"/>
+                <cylinder length="${elbow_link_length}" radius="0.04"/>
             </geometry>
-            <origin xyz="0 0 0.17" rpy="0 0 0"/>
+            <origin xyz="0 0 ${elbow_link_length/2}" rpy="0 0 0"/>
             <material name="white"/>
         </visual>
         <collision>
             <geometry>
-                <cylinder length="0.34" radius="0.04"/>
+                <cylinder length="${elbow_link_length}" radius="0.04"/>
             </geometry>
-            <origin xyz="0 0 0.17" rpy="0 0 0"/>
+            <origin xyz="0 0 ${elbow_link_length/2}" rpy="0 0 0"/>
         </collision>
         <inertial>
@@ -117,19 +122,19 @@
         <child link="wrist_deviation_link"/>
         <limit effort="1000.0" lower="${M_PI/2}" upper="${M_PI*3/2}" velocity="0.5"/>
-        <origin xyz="0 0 0.34" rpy="${M_PI} 0 ${M_PI}"/>
+        <origin xyz="0 0 ${elbow_link_length}" rpy="${M_PI} 0 ${M_PI}"/>
     </joint>
     <link name="wrist_deviation_link">
         <visual>
             <geometry>
-                <cylinder length="0.10" radius="0.04"/>
+                <cylinder length="${wrist_deviation_link_length}" radius="0.04"/>
             </geometry>
-            <origin xyz="0 0 0.05" rpy="0 0 0"/>
+            <origin xyz="0 0 ${wrist_deviation_link_length/2}" rpy="0 0 0"/>
             <material name="green"/>
         </visual>
         <collision>
             <geometry>
-                <cylinder length="0.10" radius="0.04"/>
+                <cylinder length="${wrist_deviation_link_length}" radius="0.04"/>
             </geometry>
-            <origin xyz="0 0 0.5" rpy="0 0 0"/>
+            <origin xyz="0 0 ${wrist_deviation_link_length/2}" rpy="0 0 0"/>
         </collision>
         <inertial>
@@ -143,19 +148,19 @@
         <child link="wrist_extension_link"/>
         <limit effort="1000.0" lower="${M_PI/2}" upper="${M_PI*3/2}" velocity="0.5"/>
-        <origin xyz="0 0 0.1" rpy="0 ${M_PI} 0"/>
+        <origin xyz="0 0 ${wrist_deviation_link_length}" rpy="0 ${M_PI} 0"/>
     </joint>
     <link name="wrist_extension_link">
         <visual>
             <geometry>
-                <cylinder length="0.10" radius="0.04"/>
+                <cylinder length="${wrist_extension_link_length}" radius="0.04"/>
             </geometry>
-            <origin xyz="0 0 0.05" rpy="0 0 0"/>
+            <origin xyz="0 0 ${wrist_extension_link_length/2}" rpy="0 0 0"/>
             <material name="blue"/>
         </visual>
         <collision>
             <geometry>
-                <cylinder length="0.10" radius="0.04"/>
+                <cylinder length="${wrist_extension_link_length}" radius="0.04"/>
             </geometry>
-            <origin xyz="0 0 0.5" rpy="0 0 0"/>
+            <origin xyz="0 0 ${wrist_extension_link_length/2}" rpy="0 0 0"/>
         </collision>
         <inertial>
@@ -164,16 +169,3 @@
         </inertial>
     </link>
-    <!--xacro:pr2_gripper_v0 reflect="-1.0" side="" parent="wrist_extension_link"
-        screw_reduction="${4.0/1000.0}"
-        gear_ratio="${(729.0/25.0)*(22.0/16.0)}"
-        theta0="${3.6029*M_PI/180.0}"
-        phi0="${29.7089*M_PI/180.0}"
-        t0="${-0.1914/1000.0}"
-        L0="${37.5528/1000.0}"
-        h="${0.0/1000.0}"
-        a="${68.3698/1000.0}"
-        b="${43.3849/1000.0}"
-        r="${91.5/1000.0}">
-        <origin xyz="0 0 0.08" rpy="0 ${-M_PI/2} ${M_PI/2}" />
-    </xacro:pr2_gripper_v0-->
 </robot>

File: tinker_description/urdf/base/base.urdf.xacro (robot description, xacro)
@@ -8,5 +8,5 @@
     <xacro:property name="base_length" value="0.64"/>
     <xacro:property name="base_width" value="0.52"/>
-    <xacro:property name="base_height" value="0.15"/>
+    <xacro:property name="base_height" value="0.18"/>
     <xacro:property name="base_laser_x" value="0.30"/>
     <xacro:property name="base_laser_y" value="0"/>
@@ -19,5 +19,5 @@
             </geometry>
             <origin xyz="0 0 ${base_height/2}"/>
-            <material name="white"/>
+            <material name="brown"/>
         </visual>
         <collision>

File: tinker_description/urdf/body/body.urdf.xacro (robot description, xacro)
@@ -3,5 +3,5 @@
     <xacro:property name="base_height" value="0.15"/>
     <xacro:property name="pillar_x" value="0"/>
-    <xacro:property name="pillar_y" value="0.20"/>
+    <xacro:property name="pillar_y" value="0.10"/>
     <link name="pillar">
         <visual>
@@ -10,5 +10,5 @@
             </geometry>
             <origin xyz="0 0 0.5" rpy="0 0 0"/>
-            <material name="white"/>
+            <material name="orange"/>
         </visual>
         <collision>
@@ -31,5 +31,5 @@
     <xacro:include filename="$(find pr2_description)/urdf/sensors/kinect2.urdf.xacro"/>
     <xacro:kinect2_v0 name="kinect" parent="pillar">
-        <origin xyz="0 0 0.9" rpy="0 0 0"/>
+        <origin xyz="0.06 0 0.9" rpy="0 0 0"/>
     </xacro:kinect2_v0>
 </robot>

Commit message: [Add] virtual joints for moveit

File: tinker_description/robot/tinker.urdf.xacro (robot description, xacro)
@@ -10,3 +10,26 @@
     <xacro:include filename="$(find tinker_description)/urdf/body/body.urdf.xacro"/>
     <xacro:include filename="$(find tinker_description)/urdf/arm/arm.urdf.xacro"/>
+    <link name="virtual_x_link"/>
+    <joint name="virtual_x_joint" type="prismatic">
+        <parent link="virtual_x_link" />
+        <child link="virtual_y_link" />
+        <origin rpy="0 0 0" />
+        <limit lower="-1" upper="1" velocity="0.2" effort="10000"/>
+    </joint>
+    <link name="virtual_y_link"/>
+    <joint name="virtual_y_joint" type="prismatic">
+        <parent link="virtual_y_link" />
+        <child link="virtual_yaw_link" />
+        <origin rpy="0 0 0" />
+        <axis xyz="0 1 0" />
+        <limit lower="-1" upper="1" velocity="0.2" effort="10000"/>
+    </joint>
+    <link name="virtual_yaw_link"/>
+    <joint name="virtual_yaw_joint" type="continuous">
+        <parent link="virtual_yaw_link" />
+        <child link="base_link" />
+        <origin rpy="0 0 0" />
+        <axis xyz="0 0 1" />
+        <limit velocity="0.2" effort="10000"/>
+    </joint>
 </robot>

Commit message: [Change] Remove shoulder rotation joint

File: tinker_description/robot/tinker.urdf.xacro (robot description, xacro)
@@ -15,5 +15,5 @@
         <child link="virtual_y_link" />
         <origin rpy="0 0 0" />
-        <limit lower="-1" upper="1" velocity="0.2" effort="10000"/>
+        <limit lower="-1000" upper="1000" velocity="0.2" effort="10000"/>
     </joint>
     <link name="virtual_y_link"/>
@@ -23,5 +23,5 @@
         <origin rpy="0 0 0" />
         <axis xyz="0 1 0" />
-        <limit lower="-1" upper="1" velocity="0.2" effort="10000"/>
+        <limit lower="-1000" upper="1000" velocity="0.2" effort="10000"/>
     </joint>
     <link name="virtual_yaw_link"/>

File: tinker_description/urdf/arm/arm.urdf.xacro (robot description, xacro)
@@ -7,6 +7,5 @@
     <xacro:property name="shoulder_link_length" value="0.41"/>
     <xacro:property name="elbow_link_length" value="0.32"/>
-    <xacro:property name="wrist_deviation_link_length" value="0.09"/>
-    <xacro:property name="wrist_extension_link_length" value="0.10"/>
+    <xacro:property name="wrist_extension_link_length" value="0.20"/>
     <joint name="arm_origin_joint" type="fixed">
         <parent link="base_link"/>
@@ -39,9 +38,9 @@
         </inertial>
     </link>
-    <joint name="shoulder_rotation_joint" type="revolute">
-        <axis xyz="0 0 1"/>
+    <joint name="shoulder_rotation_joint" type="fixed">
+        <!--axis xyz="0 0 1"/-->
         <parent link="arm_base_link"/>
         <child link="shoulder_base_link"/>
-        <limit effort="1000.0" lower="${-M_PI/2}" upper="${M_PI/2}" velocity="0.5"/>
+        <!--limit effort="1000.0" lower="${-M_PI/2}" upper="${M_PI/2}" velocity="0.5"/-->
         <origin xyz="0 0 0" rpy="0 0 ${M_PI/2}"/>
     </joint>
@@ -117,36 +116,10 @@
         </inertial>
     </link>
-    <joint name="wrist_deviation" type="revolute">
-        <axis xyz="0 1 0"/>
-        <parent link="elbow_link"/>
-        <child link="wrist_deviation_link"/>
-        <limit effort="1000.0" lower="${M_PI/2}" upper="${M_PI*3/2}" velocity="0.5"/>
-        <origin xyz="0 0 ${elbow_link_length}" rpy="${M_PI} 0 ${M_PI}"/>
-    </joint>
-    <link name="wrist_deviation_link">
-        <visual>
-            <geometry>
-                <cylinder length="${wrist_deviation_link_length}" radius="0.04"/>
-            </geometry>
-            <origin xyz="0 0 ${wrist_deviation_link_length/2}" rpy="0 0 0"/>
-            <material name="green"/>
-        </visual>
-        <collision>
-            <geometry>
-                <cylinder length="${wrist_deviation_link_length}" radius="0.04"/>
-            </geometry>
-            <origin xyz="0 0 ${wrist_deviation_link_length/2}" rpy="0 0 0"/>
-        </collision>
-        <inertial>
-            <mass value="1"/>
-            <inertia ixx="0.0" ixy="0.0" ixz="0.0" iyy="0.0" iyz="0.0" izz="0.0"/>
-        </inertial>
-    </link>
     <joint name="wrist_extension" type="revolute">
         <axis xyz="1 0 0"/>
-        <parent link="wrist_deviation_link"/>
+        <parent link="elbow_link"/>
         <child link="wrist_extension_link"/>
         <limit effort="1000.0" lower="${M_PI/2}" upper="${M_PI*3/2}" velocity="0.5"/>
-        <origin xyz="0 0 ${wrist_deviation_link_length}" rpy="0 ${M_PI} 0"/>
+        <origin xyz="0 0 ${elbow_link_length}" rpy="0 ${M_PI} 0"/>
     </joint>
     <link name="wrist_extension_link">
