Commit message: [Add] Gazebo ros_control config for tinker

File: tinker_description/robot/tinker.urdf.xacro (robot description, xacro)
@@ -10,26 +10,4 @@
     <xacro:include filename="$(find tinker_description)/urdf/body/body.urdf.xacro"/>
     <xacro:include filename="$(find tinker_description)/urdf/arm/arm.urdf.xacro"/>
-    <link name="virtual_x_link"/>
-    <joint name="virtual_x_joint" type="prismatic">
-        <parent link="virtual_x_link" />
-        <child link="virtual_y_link" />
-        <origin rpy="0 0 0" />
-        <limit lower="-1000" upper="1000" velocity="0.2" effort="10000"/>
-    </joint>
-    <link name="virtual_y_link"/>
-    <joint name="virtual_y_joint" type="prismatic">
-        <parent link="virtual_y_link" />
-        <child link="virtual_yaw_link" />
-        <origin rpy="0 0 0" />
-        <axis xyz="0 1 0" />
-        <limit lower="-1000" upper="1000" velocity="0.2" effort="10000"/>
-    </joint>
-    <link name="virtual_yaw_link"/>
-    <joint name="virtual_yaw_joint" type="continuous">
-        <parent link="virtual_yaw_link" />
-        <child link="base_link" />
-        <origin rpy="0 0 0" />
-        <axis xyz="0 0 1" />
-        <limit velocity="0.2" effort="10000"/>
-    </joint>
+    <xacro:include filename="$(find tinker_description)/robot/tinker.gazebo.xacro"/>
 </robot>

File: tinker_description/urdf/arm/arm.urdf.xacro (robot description, xacro)
@@ -13,5 +13,10 @@
         <origin xyz="${arm_origin_x} ${arm_origin_y} ${arm_origin_z}" rpy="0 0 0"/>
     </joint>
-    <link name="arm_origin_link"/>
+    <link name="arm_origin_link">
+        <inertial>
+            <mass value="1"/>
+            <inertia ixx="0.1" ixy="0.1" ixz="0.1" iyy="0.1" iyz="0.1" izz="0.1"/>
+        </inertial>
+    </link>
     <joint name="arm_base_joint" type="prismatic">
         <axis xyz="0 0 1"/>
@@ -35,5 +40,5 @@
         <inertial>
             <mass value="1"/>
-            <inertia ixx="0.0" ixy="0.0" ixz="0.0" iyy="0.0" iyz="0.0" izz="0.0"/>
+            <inertia ixx="0.1" ixy="0.1" ixz="0.1" iyy="0.1" iyz="0.1" izz="0.1"/>
         </inertial>
     </link>
@@ -61,5 +66,5 @@
         <inertial>
             <mass value="1"/>
-            <inertia ixx="0.0" ixy="0.0" ixz="0.0" iyy="0.0" iyz="0.0" izz="0.0"/>
+            <inertia ixx="0.1" ixy="0.1" ixz="0.1" iyy="0.1" iyz="0.1" izz="0.1"/>
         </inertial>
     </link>
@@ -87,5 +92,5 @@
         <inertial>
             <mass value="1"/>
-            <inertia ixx="0.0" ixy="0.0" ixz="0.0" iyy="0.0" iyz="0.0" izz="0.0"/>
+            <inertia ixx="0.1" ixy="0.1" ixz="0.1" iyy="0.1" iyz="0.1" izz="0.1"/>
         </inertial>
     </link>
@@ -113,5 +118,5 @@
         <inertial>
             <mass value="1"/>
-            <inertia ixx="0.0" ixy="0.0" ixz="0.0" iyy="0.0" iyz="0.0" izz="0.0"/>
+            <inertia ixx="0.1" ixy="0.1" ixz="0.1" iyy="0.1" iyz="0.1" izz="0.1"/>
         </inertial>
     </link>
@@ -139,5 +144,5 @@
         <inertial>
             <mass value="1"/>
-            <inertia ixx="0.0" ixy="0.0" ixz="0.0" iyy="0.0" iyz="0.0" izz="0.0"/>
+            <inertia ixx="0.1" ixy="0.1" ixz="0.1" iyy="0.1" iyz="0.1" izz="0.1"/>
         </inertial>
     </link>

File: tinker_description/urdf/base/base.gazebo.xacro (robot description, xacro)
@@ -4,12 +4,3 @@
         <material>Gazebo/White</material>
     </gazebo>
-    <gazebo>
-        <plugin name="object_controller" filename="libgazebo_ros_planar_move.so">
-            <commandTopic>cmd_vel</commandTopic>
-            <odometryTopic>odom</odometryTopic>
-            <odometryFrame>odom</odometryFrame>
-            <odometryRate>20.0</odometryRate>
-            <robotBaseFrame>base_link</robotBaseFrame>
-        </plugin>
-    </gazebo>
 </robot>

File: tinker_description/urdf/base/base.urdf.xacro (robot description, xacro)
@@ -20,4 +20,42 @@
     <xacro:property name="back_xtion_z" value="0.1"/>
     <!--*****************chasiss***********************-->
+    <link name="virtual_x_link">
+        <inertial>
+            <mass value="1"/>
+            <inertia ixx="0.1" ixy="0.1" ixz="0.1" iyy="0.1" iyz="0.1" izz="0.1"/>
+        </inertial>
+    </link>
+    <joint name="virtual_x_joint" type="prismatic">
+        <parent link="virtual_x_link" />
+        <child link="virtual_y_link" />
+        <origin rpy="0 0 0" />
+        <limit lower="-1000" upper="1000" velocity="0.2" effort="10000"/>
+    </joint>
+    <link name="virtual_y_link">
+        <inertial>
+            <mass value="1"/>
+            <inertia ixx="0.1" ixy="0.1" ixz="0.1" iyy="0.1" iyz="0.1" izz="0.1"/>
+        </inertial>
+    </link>
+    <joint name="virtual_y_joint" type="prismatic">
+        <parent link="virtual_y_link" />
+        <child link="virtual_yaw_link" />
+        <origin rpy="0 0 0" />
+        <axis xyz="0 1 0" />
+        <limit lower="-1000" upper="1000" velocity="0.2" effort="10000"/>
+    </joint>
+    <link name="virtual_yaw_link">
+        <inertial>
+            <mass value="1"/>
+            <inertia ixx="0.1" ixy="0.1" ixz="0.1" iyy="0.1" iyz="0.1" izz="0.1"/>
+        </inertial>
+    </link>
+    <joint name="virtual_yaw_joint" type="continuous">
+        <parent link="virtual_yaw_link" />
+        <child link="base_link" />
+        <origin rpy="0 0 0" />
+        <axis xyz="0 0 1" />
+        <limit velocity="0.2" effort="10000"/>
+    </joint>
     <link name="base_link">
         <visual>
@@ -37,5 +75,5 @@
             <origin xyz="0 0 ${base_height/2}"/>
             <mass value="1"/>
-            <inertia ixx="0.0" ixy="0.0" ixz="0.0" iyy="0.0" iyz="0.0" izz="0.0"/>
+            <inertia ixx="0.1" ixy="0.1" ixz="0.1" iyy="0.1" iyz="0.1" izz="0.1"/>
         </inertial>
     </link>

File: tinker_description/urdf/body/body.urdf.xacro (robot description, xacro)
@@ -20,5 +20,5 @@
         <inertial>
             <mass value="1"/>
-            <inertia ixx="0.0" ixy="0.0" ixz="0.0" iyy="0.0" iyz="0.0" izz="0.0"/>
+            <inertia ixx="0.1" ixy="0.1" ixz="0.1" iyy="0.1" iyz="0.1" izz="0.1"/>
             <origin xyz="0 0 0.5" rpy="0 0 0"/>
         </inertial>
